Commit message: Add files via upload

File: my_robot_description/urdf/robot.urdf (robot description, URDF)
Before this commit: robot robotModel, 14 links, 13 joints
Links:
- link base: geometry collision mesh filename=package://my_robot_description/meshes/base.stl; visual mesh filename=package://my_robot_description/meshes/base.stl
- link part_1: geometry collision mesh filename=package://my_robot_description/meshes/part_1.stl; visual mesh filename=package://my_robot_description/meshes/part_1.stl
- link part_1_10: geometry collision mesh filename=package://my_robot_description/meshes/part_1.stl; visual mesh filename=package://my_robot_description/meshes/part_1.stl
- link part_1_11: geometry collision mesh filename=package://my_robot_description/meshes/part_1.stl; visual mesh filename=package://my_robot_description/meshes/part_1.stl
- link part_1_12: geometry collision mesh filename=package://my_robot_description/meshes/part_1.stl; visual mesh filename=package://my_robot_description/meshes/part_1.stl
- link part_1_2: geometry collision mesh filename=package://my_robot_description/meshes/part_1.stl; visual mesh filename=package://my_robot_description/meshes/part_1.stl
- link part_1_3: geometry collision mesh filename=package://my_robot_description/meshes/part_1.stl; visual mesh filename=package://my_robot_description/meshes/part_1.stl
- link part_1_4: geometry collision mesh filename=package://my_robot_description/meshes/part_1.stl; visual mesh filename=package://my_robot_description/meshes/part_1.stl
- link part_1_5: geometry collision mesh filename=package://my_robot_description/meshes/part_1.stl; visual mesh filename=package://my_robot_description/meshes/part_1.stl
- link part_1_6: geometry collision mesh filename=package://my_robot_description/meshes/part_1.stl; visual mesh filename=package://my_robot_description/meshes/part_1.stl
- link part_1_7: geometry collision mesh filename=package://my_robot_description/meshes/part_1.stl; visual mesh filename=package://my_robot_description/meshes/part_1.stl
- link part_1_8: geometry collision mesh filename=package://my_robot_description/meshes/part_1.stl; visual mesh filename=package://my_robot_description/meshes/part_1.stl
- link part_1_9: geometry collision mesh filename=package://my_robot_description/meshes/part_1.stl; visual mesh filename=package://my_robot_description/meshes/part_1.stl
